File: Quad-AMBE3000.kicad_pcb (KiCad board)
At the start: 2 copper layers, 216 parts, among them J1 USB_C, Q1 BS170F, Q2 BS170F, Q3 BS170F, Q4 BS170F, U1 74AVC9112DCH, U10 AMBE-3000R, U2 74HC595D, U3 AT93C46D-TH-T, U4 FT4232HL, U5 TPS7A8001DRBR, U6 TPS7A8001DRBR, U7 AMBE-3000R, U8 AMBE-3000R, U9 AMBE-3000R, X1 29.4912MHz, Y1 12M

Commit message: Most of the layout done
Parts:
- removed the C11 at (178.9, 124.2)
- removed the C14 at (182.9, 109.2)
- removed the C62 at (131.5, 71.8)
- removed the C63 at (131.5, 74.3)
- removed the C77 at (171.7, 72.5)
- removed the C78 at (171.7, 75.0)
- removed C92: 4u7, Capacitor_SMD:C_0603_1608Metric
- removed D10, D11, D12, D13, D14, D15, D16, D17, D18, D19, D20, D21, D22, D23, D24, D25, D9: GRN, LED_SMD:LED_0603_1608Metric
- removed FB10, FB11, FB12, FB5, FB6, FB7, FB8, FB9: 600R/100M, Inductor_SMD:L_0805_2012Metric
- removed the R23 at (190.9, 124.2)
- removed the R31 at (88.5, 79.2)
- removed the R32 at (88.5, 81.7)
- removed the R34 at (92.5, 71.7)
- removed the R35 at (92.5, 74.2)
- removed the R40 at (131.5, 79.3)
- removed the R41 at (131.5, 81.8)
- removed the R43 at (135.5, 71.8)
- removed the R44 at (135.5, 74.3)
- removed R49, R50, R52, R53, R58, R59, R61, R62: 330R, Resistor_SMD:R_0603_1608Metric
- added C109: 100n, Capacitor_SMD:C_0603_1608Metric, F.Cu at (178.2, 73.7)
- added C110: 100n, Capacitor_SMD:C_0603_1608Metric, F.Cu at (193.0, 59.9)
- added C111: 100n, Capacitor_SMD:C_0603_1608Metric, F.Cu at (197.8, 69.9)
- added C112: 100n, Capacitor_SMD:C_0603_1608Metric, F.Cu at (189.8, 59.9)
- added C114: 100n, Capacitor_SMD:C_0603_1608Metric, F.Cu at (178.2, 76.9)
- added C115: 100n, Capacitor_SMD:C_0603_1608Metric, F.Cu at (178.2, 70.5)
- added C13: 27p, Capacitor_SMD:C_0603_1608Metric, F.Cu at (129.4, 42.0)
- added C46: 100n, Capacitor_SMD:C_0603_1608Metric, F.Cu at (153.2, 38.5)
- added C49: 100n, Capacitor_SMD:C_0603_1608Metric, F.Cu at (166.2, 51.6)
- added C51: 100n, Capacitor_SMD:C_0603_1608Metric, F.Cu at (159.7, 50.7)
- added C52: 100n, Capacitor_SMD:C_0603_1608Metric, F.Cu at (153.2, 41.7)
- added C67: 100n, Capacitor_SMD:C_0603_1608Metric, F.Cu at (197.7, 38.0)
- added C68: 100n, Capacitor_SMD:C_0603_1608Metric, F.Cu at (197.7, 44.6)
- added C69: 100n, Capacitor_SMD:C_0603_1608Metric, F.Cu at (197.7, 41.4)
- added C70: 100n, Capacitor_SMD:C_0603_1608Metric, F.Cu at (184.7, 50.6)
- added C72: 100n, Capacitor_SMD:C_0603_1608Metric, F.Cu at (191.1, 51.4)
- added C73: 100n, Capacitor_SMD:C_0603_1608Metric, F.Cu at (194.7, 50.6)
- added C88: 100n, Capacitor_SMD:C_0603_1608Metric, F.Cu at (172.7, 66.7)
- added C89: 100n, Capacitor_SMD:C_0603_1608Metric, F.Cu at (168.1, 59.9)
- added C90: 100n, Capacitor_SMD:C_0603_1608Metric, F.Cu at (172.7, 69.9)
- added C91: 100n, Capacitor_SMD:C_0603_1608Metric, F.Cu at (164.9, 59.9)
- added C94: 100n, Capacitor_SMD:C_0603_1608Metric, F.Cu at (153.3, 70.3)
- added H1: M3, MountingHole:MountingHole_3.2mm_M3_Pad_Via, F.Cu at (124.0, 27.0)
- added H2: M3, MountingHole:MountingHole_3.2mm_M3_Pad_Via, F.Cu at (200.0, 27.0)
- added H3: M3, MountingHole:MountingHole_3.2mm_M3_Pad_Via, F.Cu at (124.0, 81.0)
- added H4: M3, MountingHole:MountingHole_3.2mm_M3_Pad_Via, F.Cu at (200.0, 81.0)
- C10: value 100n -> 27p
- C47, C48, C93: value 4u7 -> 100n
- moved FB4 117.9 mm to (126.1, 35.3), turned to 180 degrees
- moved Y1 117.7 mm to (130.3, 39.5)
- moved FB3 114.4 mm to (126.1, 37.3), turned to 180 degrees
- moved R14 112.1 mm to (131.8, 26.6), turned to -90 degrees
- moved R13 110.7 mm to (130.2, 26.6), turned to -90 degrees
- moved U3 110.4 mm to (141.2, 36.0)
- moved U2 109.2 mm to (141.4, 29.2), turned to -90 degrees
- moved J1 105.1 mm to (123.0, 45.3), turned to -90 degrees
- moved R12 104.9 mm to (128.6, 32.0), turned to -90 degrees
- moved R11 101.9 mm to (130.2, 32.0), turned to -90 degrees
- moved FB2 101.5 mm to (129.6, 49.3), turned to 180 degrees
- moved R20 99.7 mm to (133.4, 35.3), turned to 180 degrees
- moved R10 98.9 mm to (131.8, 32.0), turned to -90 degrees
- moved C43 98.7 mm to (172.7, 34.7), turned to -90 degrees
- moved C38 98.4 mm to (165.0, 31.3), turned to 180 degrees
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- renumbered C83 to C100, C84 to C101, C85 to C102, C86 to C103, C87 to C104, C88 to C105, C89 to C106, C90 to C107, C91 to C108, C12 to C11, C13 to C12, C15 to C14, C16 to C15, C17 to C16, C18 to C17, C19 to C18, C20 to C19, C21 to C20, C22 to C21, C23 to C22, C24 to C23, C25 to C24, C26 to C25, C27 to C26, C28 to C27, C29 to C28, C30 to C29, C31 to C30, C32 to C31, C33 to C32, C34 to C33, C35 to C34, C36 to C35, C37 to C36, C38 to C37, C39 to C38, C40 to C39, C41 to C40, C42 to C41, C43 to C42, C44 to C43, C45 to C44, C46 to C45, C49 to C54, C50 to C55, C51 to C56, C52 to C57, C53 to C58, C54 to C59, C55 to C60, C56 to C61, C57 to C62, C58 to C63, C59 to C64, C60 to C65, C61 to C66, C64 to C75, C65 to C76, C66 to C77, C67 to C78, C68 to C79, C69 to C80, C70 to C81, C71 to C82, C72 to C83, C73 to C84, C74 to C85, C75 to C86, C76 to C87, C79 to C96, C80 to C97, C81 to C98, C82 to C99, R24 to R23, R25 to R24, R26 to R25, R27 to R26, R28 to R27, R29 to R28, R30 to R29, R33 to R30, R36 to R31, R37 to R32, R38 to R33, R39 to R34, R42 to R35, R45 to R36, R46 to R37, R47 to R38, R48 to R39, R51 to R40, R54 to R41, R55 to R42, R56 to R43, R57 to R44, R60 to R45, R63 to R46, R64 to R47, R65 to R48
Connections:
- net /USB & UART Interface/USB_Dm renamed /USB & UART Interface/USB_D-
- net /USB & UART Interface/USB_Dp renamed /USB & UART Interface/USB_D+
- net Net-(U1-VCC) renamed /3V3_OSC
- C10 pad 2: /USB & UART Interface/FTDI_1V8 -> Net-(U4-OSCI)
- C101 pad 2: Net-(C81-Pad2) -> +1V8
- C102 pad 2: Net-(C82-Pad2) -> +3V3
- C103 pad 2: Net-(C81-Pad2) -> +1V8
- C104 pad 2: Net-(C82-Pad2) -> +3V3
- C106 pad 2: Net-(C81-Pad2) -> +1V8
- C107 pad 2: Net-(C82-Pad2) -> +3V3
- C108 pad 2: Net-(C81-Pad2) -> +1V8
- C35 pad 2: Net-(C36-Pad2) -> +1V8
- C36 pad 2: Net-(C37-Pad2) -> +3V3
- C38 pad 2: Net-(C36-Pad2) -> +1V8
- C39 pad 2: Net-(C37-Pad2) -> +3V3
- C40 pad 2: Net-(C36-Pad2) -> +1V8
- C41 pad 2: Net-(C37-Pad2) -> +3V3
- C43 pad 2: Net-(C36-Pad2) -> +1V8
- C44 pad 2: Net-(C37-Pad2) -> +3V3
- C45 pad 2: Net-(C36-Pad2) -> +1V8
- C47 pad 2: Net-(C37-Pad2) -> +1V8
- C48 pad 2: Net-(C36-Pad2) -> +3V3
- C56 pad 2: Net-(C51-Pad2) -> +1V8
- C57 pad 2: Net-(C52-Pad2) -> +3V3
- C59 pad 2: Net-(C51-Pad2) -> +1V8
- C60 pad 2: Net-(C52-Pad2) -> +3V3
- C61 pad 2: Net-(C51-Pad2) -> +1V8
- C62 pad 2: Net-(C52-Pad2) -> +3V3
- C64 pad 2: Net-(C51-Pad2) -> +1V8
- C65 pad 2: Net-(C52-Pad2) -> +3V3
- C66 pad 2: Net-(C51-Pad2) -> +1V8
- C77 pad 2: Net-(C66-Pad2) -> +1V8
- C78 pad 2: Net-(C67-Pad2) -> +3V3
- C80 pad 2: Net-(C66-Pad2) -> +1V8
- C81 pad 2: Net-(C67-Pad2) -> +3V3
- C82 pad 2: Net-(C66-Pad2) -> +1V8
- C83 pad 2: Net-(C67-Pad2) -> +3V3
- C85 pad 2: Net-(C66-Pad2) -> +1V8
- C86 pad 2: Net-(C67-Pad2) -> +3V3
- C87 pad 2: Net-(C66-Pad2) -> +1V8
- C93 pad 2: Net-(C81-Pad2) -> +1V8
- C98 pad 2: Net-(C81-Pad2) -> +1V8
- C99 pad 2: Net-(C82-Pad2) -> +3V3
- J1 pad A8: (no net) -> unconnected-(J1-SBU1-PadA8)
- J1 pad B8: (no net) -> unconnected-(J1-SBU2-PadB8)
- R33 pad 2: Net-(C37-Pad2) -> +3V3
- R38 pad 2: Net-(C52-Pad2) -> +3V3
- R43 pad 2: Net-(C67-Pad2) -> +3V3
- R48 pad 2: Net-(C82-Pad2) -> +3V3
- U10 pad 1: Net-(C82-Pad2) -> +3V3
- U10 pad 102: Net-(C81-Pad2) -> +1V8
- U10 pad 104: Net-(C82-Pad2) -> +3V3
- U10 pad 110: Net-(C81-Pad2) -> +1V8
- U10 pad 114: Net-(C81-Pad2) -> +1V8
- U10 pad 118: Net-(C82-Pad2) -> +3V3
- U10 pad 13: Net-(C82-Pad2) -> +3V3
- U10 pad 14: Net-(C82-Pad2) -> +3V3
- U10 pad 20: Net-(C81-Pad2) -> +1V8
- U10 pad 25: Net-(C82-Pad2) -> +3V3
- U10 pad 29: Net-(C81-Pad2) -> +1V8
- U10 pad 42: Net-(C81-Pad2) -> +1V8
- U10 pad 44: Net-(D22-K) -> unconnected-(U10A-STANDBYn-Pad44)
- U10 pad 45: Net-(D23-K) -> unconnected-(U10A-IDLEn-Pad45)
- U10 pad 49: Net-(C82-Pad2) -> +3V3
- U10 pad 56: Net-(C81-Pad2) -> +1V8
- U10 pad 61: Net-(D24-K) -> unconnected-(U10A-RUNn-Pad61)
- U10 pad 63: Net-(C81-Pad2) -> +1V8
- U10 pad 69: Net-(D25-A) -> unconnected-(U10A-TX_RDY-Pad69)
- U10 pad 74: Net-(C81-Pad2) -> +1V8
- U10 pad 75: Net-(U10A-STDBY_ENABLEn) -> unconnected-(U10A-STDBY_ENABLEn-Pad75)
- U10 pad 82: Net-(C81-Pad2) -> +1V8
- U10 pad 83: Net-(C82-Pad2) -> +3V3
- U10 pad 94: Net-(C81-Pad2) -> +1V8
- U4 pad 60: Net-(D9-K) -> /USB & UART Interface/FTDI_PWREN
- U7 pad 1: Net-(C37-Pad2) -> +3V3
- U7 pad 102: Net-(C36-Pad2) -> +1V8
- U7 pad 104: Net-(C37-Pad2) -> +3V3
- U7 pad 110: Net-(C36-Pad2) -> +1V8
- U7 pad 114: Net-(C36-Pad2) -> +1V8
- U7 pad 118: Net-(C37-Pad2) -> +3V3
- U7 pad 13: Net-(C37-Pad2) -> +3V3
- U7 pad 14: Net-(C37-Pad2) -> +3V3
- U7 pad 20: Net-(C36-Pad2) -> +1V8
- U7 pad 25: Net-(C37-Pad2) -> +3V3
- U7 pad 29: Net-(C36-Pad2) -> +1V8
- U7 pad 42: Net-(C36-Pad2) -> +1V8
- U7 pad 44: Net-(D10-K) -> unconnected-(U7A-STANDBYn-Pad44)
- U7 pad 45: Net-(D11-K) -> unconnected-(U7A-IDLEn-Pad45)
- U7 pad 49: Net-(C37-Pad2) -> +3V3
- U7 pad 56: Net-(C36-Pad2) -> +1V8
- U7 pad 61: Net-(D12-K) -> unconnected-(U7A-RUNn-Pad61)
- U7 pad 63: Net-(C36-Pad2) -> +1V8
- U7 pad 69: Net-(D13-A) -> unconnected-(U7A-TX_RDY-Pad69)
- U7 pad 74: Net-(C36-Pad2) -> +1V8
- U7 pad 75: Net-(U7A-STDBY_ENABLEn) -> unconnected-(U7A-STDBY_ENABLEn-Pad75)
- U7 pad 82: Net-(C36-Pad2) -> +1V8
- U7 pad 83: Net-(C37-Pad2) -> +3V3
- U7 pad 94: Net-(C36-Pad2) -> +1V8
- U8 pad 1: Net-(C52-Pad2) -> +3V3
- U8 pad 102: Net-(C51-Pad2) -> +1V8
- U8 pad 104: Net-(C52-Pad2) -> +3V3
- U8 pad 110: Net-(C51-Pad2) -> +1V8
- U8 pad 114: Net-(C51-Pad2) -> +1V8
- U8 pad 118: Net-(C52-Pad2) -> +3V3
- U8 pad 13: Net-(C52-Pad2) -> +3V3
- U8 pad 14: Net-(C52-Pad2) -> +3V3
- U8 pad 20: Net-(C51-Pad2) -> +1V8
- U8 pad 25: Net-(C52-Pad2) -> +3V3
- U8 pad 29: Net-(C51-Pad2) -> +1V8
- U8 pad 42: Net-(C51-Pad2) -> +1V8
- U8 pad 44: Net-(D14-K) -> unconnected-(U8A-STANDBYn-Pad44)
- U8 pad 45: Net-(D15-K) -> unconnected-(U8A-IDLEn-Pad45)
- U8 pad 49: Net-(C52-Pad2) -> +3V3
- U8 pad 56: Net-(C51-Pad2) -> +1V8
- U8 pad 61: Net-(D16-K) -> unconnected-(U8A-RUNn-Pad61)
- U8 pad 63: Net-(C51-Pad2) -> +1V8
- U8 pad 69: Net-(D17-A) -> unconnected-(U8A-TX_RDY-Pad69)
- U8 pad 74: Net-(C51-Pad2) -> +1V8
- U8 pad 75: Net-(U8A-STDBY_ENABLEn) -> unconnected-(U8A-STDBY_ENABLEn-Pad75)
- U8 pad 82: Net-(C51-Pad2) -> +1V8
- U8 pad 83: Net-(C52-Pad2) -> +3V3
- U8 pad 94: Net-(C51-Pad2) -> +1V8
- U9 pad 1: Net-(C67-Pad2) -> +3V3
- U9 pad 102: Net-(C66-Pad2) -> +1V8
- U9 pad 104: Net-(C67-Pad2) -> +3V3
- U9 pad 110: Net-(C66-Pad2) -> +1V8
- U9 pad 114: Net-(C66-Pad2) -> +1V8
- U9 pad 118: Net-(C67-Pad2) -> +3V3
- U9 pad 13: Net-(C67-Pad2) -> +3V3
- U9 pad 14: Net-(C67-Pad2) -> +3V3
- U9 pad 20: Net-(C66-Pad2) -> +1V8
- U9 pad 25: Net-(C67-Pad2) -> +3V3
- U9 pad 29: Net-(C66-Pad2) -> +1V8
- U9 pad 42: Net-(C66-Pad2) -> +1V8
- U9 pad 44: Net-(D18-K) -> unconnected-(U9A-STANDBYn-Pad44)
- U9 pad 45: Net-(D19-K) -> unconnected-(U9A-IDLEn-Pad45)
- U9 pad 49: Net-(C67-Pad2) -> +3V3
- U9 pad 56: Net-(C66-Pad2) -> +1V8
- U9 pad 61: Net-(D20-K) -> unconnected-(U9A-RUNn-Pad61)
- U9 pad 63: Net-(C66-Pad2) -> +1V8
- U9 pad 69: Net-(D21-A) -> unconnected-(U9A-TX_RDY-Pad69)
- U9 pad 74: Net-(C66-Pad2) -> +1V8
- U9 pad 75: Net-(U9A-STDBY_ENABLEn) -> unconnected-(U9A-STDBY_ENABLEn-Pad75)
- U9 pad 82: Net-(C66-Pad2) -> +1V8
- U9 pad 83: Net-(C67-Pad2) -> +3V3
- U9 pad 94: Net-(C66-Pad2) -> +1V8
- Y1 pad 1: Net-(U4-OSCI) -> Net-(U4-OSCO)
- Y1 pad 3: Net-(U4-OSCO) -> Net-(U4-OSCI)
Routing:
- net +1V8: track 0.00 -> 139.8 mm, vias 0 -> 44
- net +3V3: track 0.00 -> 136.1 mm, vias 0 -> 53
- net GND: track 0.00 -> 31.8 mm, vias 0 -> 51
- net /USB & UART Interface/FTDI_PWREN: track 0.00 -> 22.8 mm
- net /USB & UART Interface/FTDI_EE_CS: track 0.00 -> 21.4 mm, vias 0 -> 2
- net /USB & UART Interface/FTDI_EE_CLK: track 0.00 -> 20.2 mm, vias 0 -> 2
- net Net-(U2-QD): track 0.00 -> 17.4 mm
- net Net-(U2-QC): track 0.00 -> 17.3 mm
- net Net-(U2-QB): track 0.00 -> 17.3 mm
- net /USB & UART Interface/FTDI_VPLL: track 0.00 -> 17.2 mm, vias 0 -> 2
- net /AMBE-3000R-B/AMBE_UART_RX: track 0.00 -> 16.3 mm
- net /AMBE-3000R-D/AMBE_UART_RX: track 0.00 -> 16.3 mm
- net /AMBE-3000R-C/AMBE_UART_RX: track 0.00 -> 16.3 mm
- net /AMBE-3000R-A/AMBE_UART_RX: track 0.00 -> 16.3 mm
- net /USB & UART Interface/FTDI_EE_DTA: track 0.00 -> 16.2 mm
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- added copper zone on In2.Cu, net +1V8
- added copper zone on In2.Cu, net +3V3
- added copper zone on In2.Cu, net /3V3_OSC
- added copper zone on F.Cu, net /USB & UART Interface/FTDI_1V8
- added copper zone on In2.Cu, net /USB & UART Interface/FTDI_1V8
- added copper zone on F.Cu, net GND
- added copper zone on In1.Cu, net GND
Other:
- board outline added: 84 x 62 mm
- copper layers 2 -> 4
- board text added: "1V8"
- board text added: "3V3"
- board text added: "A"
- board text added: "B"
- board text added: "C"
- board text added: "D"
- board text added: "{ "ViaStitching": "0.2", "stitch_zone_0": { "HSpacing": "0.5", "VSpacing": "0.25", "Clearance": "0", "Randomize": false } }"
- board text added: "{ "ViaStitching": "0.2", "stitch_zone_0": { "HSpacing": "1", "VSpacing": "1", "Clearance": "0", "Randomize": false } }"
