File: ambe-vocoder.kicad_sch (KiCad schematic)
At the start: 18 parts, among them Q2 BS170F, U9 AMBE-3000R

Commit message: Schematic V1 done
Parts:
- added C36, C37, C39, C40, C41, C42, C43, C44, C45, C46: 100n, Capacitor_SMD:C_0603_1608Metric, symbol Device:C_Small
- added C47, C48: 4u7, Capacitor_SMD:C_0603_1608Metric, symbol Device:C_Small
- added FB5, FB6: 600R/100M, Inductor_SMD:L_0805_2012Metric, symbol Device:FerriteBead_Small
- added R38: 5R1, Resistor_SMD:R_0603_1608Metric, symbol Device:R_Small
- C34: renamed from C61; footprint (none) -> Capacitor_SMD:C_0603_1608Metric
- C35: renamed from C62; footprint (none) -> Capacitor_SMD:C_0603_1608Metric
- C38: renamed from C63; footprint (none) -> Capacitor_SMD:C_0603_1608Metric
- D10: renamed from D12; footprint (none) -> LED_SMD:LED_0603_1608Metric
- D11: renamed from D13; footprint (none) -> LED_SMD:LED_0603_1608Metric
- D12: renamed from D14; footprint (none) -> LED_SMD:LED_0603_1608Metric
- D13: renamed from D15; footprint (none) -> LED_SMD:LED_0603_1608Metric
- R30: renamed from R57; footprint (none) -> Resistor_SMD:R_0603_1608Metric
- R31: renamed from R58; footprint (none) -> Resistor_SMD:R_0603_1608Metric
- R32: renamed from R59; footprint (none) -> Resistor_SMD:R_0603_1608Metric
- R33: renamed from R56; footprint (none) -> Resistor_SMD:R_0603_1608Metric
- R34: renamed from R60; footprint (none) -> Resistor_SMD:R_0603_1608Metric
- R35: renamed from R61; footprint (none) -> Resistor_SMD:R_0603_1608Metric
- R36: renamed from R55; footprint (none) -> Resistor_SMD:R_0603_1608Metric
- R37: renamed from R54; footprint (none) -> Resistor_SMD:R_0603_1608Metric
- U7: renamed from U9; LCSC (none) -> DNF
- renumbered Q2 to Q1
Connections:
- net +1V8: now also FB5.1; no longer U7.102 (VDDCORE), U7.110 (VDDCORE), U7.114 (VDDCORE), U7.20 (VDDCORE), U7.29 (VDDCORE), U7.42 (VDDCORE), U7.56 (VDDCORE), U7.63 (VDDCORE), U7.74 (VDDCORE), U7.82 (VDDCORE), U7.94 (VDDCORE)
- net +3V3: now also FB6.1; no longer U7.1 (VDDIO), U7.104 (VDDIO), U7.118 (VDDIO), U7.13 (VDDIO), U7.14 (VDDIO), U7.25 (VDDIO), U7.49 (VDDIO), U7.52 (3v3FL), U7.83 (VDDIO)
- net GND: now also C36.1, C37.1, C39.1, C40.1, C41.1, C42.1, C43.1, C44.1, C45.1, C46.1, C47.1, C48.1
- new net: C37.2, C40.2, C42.2, C45.2, C47.2, FB6.2, R38.2, U7.1 (VDDIO), U7.104 (VDDIO), U7.118 (VDDIO), U7.13 (VDDIO), U7.14 (VDDIO), U7.25 (VDDIO), U7.49 (VDDIO), U7.83 (VDDIO)
- new net: C36.2, C39.2, C41.2, C44.2, C46.2, C48.2, FB5.2, U7.102 (VDDCORE), U7.110 (VDDCORE), U7.114 (VDDCORE), U7.20 (VDDCORE), U7.29 (VDDCORE), U7.42 (VDDCORE), U7.56 (VDDCORE), U7.63 (VDDCORE), U7.74 (VDDCORE), U7.82 (VDDCORE), U7.94 (VDDCORE)
- new net: C43.2, R38.1, U7.52 (3v3FL)
Other:
- note added: "Flash Supply No idea why it's filtered, but everyone does it!"
- note added: "When designing a system using the UART interface on the AMBE-3000 Vocoder Chip it is necessary that the UART_TX pin (pin 111 QFP - pin C7 BGA) be held high at boot. This will ensure the AMBE-3000 Vocoder Chip will start in the proper configuration"
- note removed: "When designing a system using the UART interface on the AMBE-3000™ Vocoder Chip it is necessary that the UART_TX pin (pin 111 QFP - pin C7 BGA) be held high at boot. This will ensure the AMBE-3000™ Vocoder Chip will start in the proper configuration"
- company: (none) -> M1GEO & G8OCV
- title: (none) -> Quad AMBE-3000R Board
- moved on the sheet: C34, C35, C38, JP1, Q1, R33, R36, R37, U7B

Commit message: Most of the layout done
Parts:
- removed D10, D11, D12, D13: GRN, LED_SMD:LED_0603_1608Metric, symbol Device:LED
- removed FB5, FB6: 600R/100M, Inductor_SMD:L_0805_2012Metric, symbol Device:FerriteBead_Small
- removed R31, R32, R34, R35: 330R, Resistor_SMD:R_0603_1608Metric, symbol Device:R_Small
- added C46, C49, C51, C52: 100n, Capacitor_SMD:C_0603_1608Metric, symbol Device:C_Small
- C47, C48: value 4u7 -> 100n
- renumbered C34 to C33, C35 to C34, C36 to C35, C37 to C36, C38 to C37, C39 to C38, C40 to C39, C41 to C40, C42 to C41, C43 to C42, C44 to C43, C45 to C44, C46 to C45, R30 to R29, R33 to R30, R36 to R31, R37 to R32, R38 to R33
Connections:
- net +1V8: now also C35.2, C38.2, C40.2, C43.2, C45.2, C47.2, U7.102 (VDDCORE), U7.110 (VDDCORE), U7.114 (VDDCORE), U7.20 (VDDCORE), U7.29 (VDDCORE), U7.42 (VDDCORE), U7.56 (VDDCORE), U7.63 (VDDCORE), U7.74 (VDDCORE), U7.82 (VDDCORE), U7.94 (VDDCORE), C49.2, C51.2, C52.2
- net +3V3: now also C36.2, C39.2, C41.2, C44.2, C48.2, R33.2, U7.1 (VDDIO), U7.104 (VDDIO), U7.118 (VDDIO), U7.13 (VDDIO), U7.14 (VDDIO), U7.25 (VDDIO), U7.49 (VDDIO), U7.83 (VDDIO), C46.2
- net GND: now also C46.1, C49.1, C51.1, C52.1
- no-connect marks 35 -> 40

Commit message: Final updates before manufacture of V1.00
Parts:
- removed Q1: BS170F, Package_TO_SOT_SMD:SOT-23, symbol Transistor_FET:BS170F
- added Q1: AO3400A, Package_TO_SOT_SMD:SOT-23, symbol Transistor_FET:AO3400A
- C33, C34, C37: LCSC (none) -> C19702
- C35, C36, C38, C39, C40, C41, C42, C43, C44, C45, C46, C47, C48, C49, C51, C52: LCSC (none) -> C14663
- JP1: footprint Jumper:SolderJumper-2_P1.3mm_Bridged_RoundedPad1.0x1.5mm -> Jumper:SolderJumper-2_P1.3mm_Open_RoundedPad1.0x1.5mm; LCSC (none) -> DNF
- R29, R30, R31: LCSC (none) -> C25804
- R32: LCSC (none) -> C25962
- R33: LCSC (none) -> C25197
Connections:
- net AMBE_UART_DTR: now also Q1.1 (G)
- net GND: now also Q1.2 (S)
- net at JP1.1 (A): now also Q1.3 (D)
Other:
- title: Quad AMBE-3000R Board -> Quad AMBE-3000R Board (AMBE-3000R Vocoder)
